Commit message: Ad Boxtra PROTO showing in Webots world, dismembered and gargantuan

File: urdf/ad_boxtra/Rover_2022.urdf (robot description, URDF)
Before this commit: robot Rover_2022, 5 links, 4 joints
Links:
- link Chassis: geometry collision mesh filename=./meshes/Chassis.STL; visual mesh filename=./meshes/Chassis.STL
- link LeftBogie: geometry collision mesh filename=./meshes/LeftBogie.STL; visual mesh filename=./meshes/LeftBogie.STL
- link LeftRocker: geometry collision mesh filename=./meshes/LeftRocker.STL; visual mesh filename=./meshes/LeftRocker.STL
- link RightBogie: geometry collision mesh filename=./meshes/RightBogie.STL; visual mesh filename=./meshes/RightBogie.STL
- link RightRocker: geometry collision mesh filename=./meshes/RightRocker.STL; visual mesh filename=./meshes/RightRocker.STL
